Commit message: urdf modifications

File: src/callisto_description/urdf/callisto.xacro (robot description, xacro)
@@ -1,4 +1,4 @@
 <?xml version='1.0'?>
-<robot name="myrobot" xmlns:xacro="http://www.ros.org/wiki/xacro">
+<robot name="callisto" xmlns:xacro="http://www.ros.org/wiki/xacro">
   <xacro:include filename="$(find callisto_description)/urdf/callisto.gazebo" />
   <xacro:include filename="$(find callisto_description)/urdf/materials.xacro" />
@@ -49,4 +49,68 @@
     </visual>
   </link>
+  <link name="fleft_wheel">
+    <!--origin xyz="-0.1 0.13 0.1" rpy="0 1.5707 1.5707"/-->
+    <collision name="collision">
+      <origin xyz="0 0 0" rpy="0 1.5707 1.5707"/>
+      <geometry>
+        <cylinder radius="0.1" length="0.05"/>
+      </geometry>
+    </collision>
+    <visual name="fleft_wheel_visual">
+      <origin xyz="0 0 0" rpy="0 1.5707 1.5707"/>
+      <geometry>
+        <cylinder radius="0.1" length="0.05"/>
+      </geometry>
+    </visual>
+    <inertial>
+      <origin xyz="0 0 0" rpy="0 1.5707 1.5707"/>
+      <mass value="5"/>
+      <cylinder_inertia m="5" r="0.1" h="0.05"/>
+      <inertia
+        ixx="1.0" ixy="0.0" ixz="0.0"
+        iyy="1.0" iyz="0.0"
+        izz="1.0"/>
+    </inertial>
+  </link>
+  <link name="fright_wheel">
+    <!--origin xyz="-0.1 -0.13 0.1" rpy="0 1.5707 1.5707"/-->
+    <collision name="collision">
+      <origin xyz="0 0 0" rpy="0 1.5707 1.5707"/>
+      <geometry>
+        <cylinder radius="0.1" length="0.05"/>
+      </geometry>
+    </collision>
+    <visual name="fright_wheel_visual">
+      <origin xyz="0 0 0" rpy="0 1.5707 1.5707"/>
+      <geometry>
+        <cylinder radius="0.1" length="0.05"/>
+      </geometry>
+    </visual>
+    <inertial>
+      <origin xyz="0 0 0" rpy="0 1.5707 1.5707"/>
+      <mass value="5"/>
+      <cylinder_inertia m="5" r="0.1" h="0.05"/>
+      <inertia
+        ixx="1.0" ixy="0.0" ixz="0.0"
+        iyy="1.0" iyz="0.0"
+        izz="1.0"/>
+    </inertial>
+  </link>
+  <joint type="continuous" name="fleft_wheel_hinge">
+    <origin xyz="-0.1 0.15 0" rpy="0 0 0"/>
+    <child link="fleft_wheel"/>
+    <parent link="chassis"/>
+    <axis xyz="0 1 0" rpy="0 0 0"/>
+    <limit effort="100" velocity="100"/>
+    <joint_properties damping="0.0" friction="0.0"/>
+  </joint>
+  <joint type="continuous" name="fright_wheel_hinge">
+    <origin xyz="-0.1 -0.15 0" rpy="0 0 0"/>
+    <child link="fright_wheel"/>
+    <parent link="chassis"/>
+    <axis xyz="0 1 0" rpy="0 0 0"/>
+    <limit effort="100" velocity="100"/>
+    <joint_properties damping="0.0" friction="0.0"/>
+  </joint>
   <link name="left_wheel">
     <!--origin xyz="0.1 0.13 0.1" rpy="0 1.5707 1.5707"/-->

Commit message: Got tf transform working - wheels weren't touching the ground

File: src/callisto_description/urdf/callisto.xacro (robot description, xacro)
@@ -17,5 +17,5 @@
     <collision name='collision'>
       <geometry>
-        <box size=".4 .2 .1"/>
+        <box size=".4 .2 .05"/>
       </geometry>
     </collision>
@@ -26,27 +26,5 @@
       </geometry>
     </visual>
-    <collision name='caster_collision'>
-      <origin xyz="-0.15 0 -0.05" rpy=" 0 0 0"/>
-      <geometry>
-        <sphere radius="0.05"/>
-      </geometry>
-      <surface>
-        <friction>
-          <ode>
-            <mu>0</mu>
-            <mu2>0</mu2>
-            <slip1>1.0</slip1>
-            <slip2>1.0</slip2>
-          </ode>
-        </friction>
-      </surface>
-    </collision>
-    <visual name='caster_visual'>
-      <origin xyz="-0.15 0 -0.05" rpy=" 0 0 0"/>
-      <geometry>
-        <sphere radius="0.05"/>
-      </geometry>
-    </visual>
-  </link>
+    </link>
   <link name="fleft_wheel">
     <!--origin xyz="-0.1 0.13 0.1" rpy="0 1.5707 1.5707"/-->
@@ -54,5 +32,5 @@
       <origin xyz="0 0 0" rpy="0 1.5707 1.5707"/>
       <geometry>
-        <cylinder radius="0.1" length="0.05"/>
+        <cylinder radius="0.03" length="0.02"/>
       </geometry>
     </collision>
@@ -60,5 +38,5 @@
       <origin xyz="0 0 0" rpy="0 1.5707 1.5707"/>
       <geometry>
-        <cylinder radius="0.1" length="0.05"/>
+        <cylinder radius="0.03" length="0.02"/>
       </geometry>
     </visual>
@@ -66,5 +44,5 @@
       <origin xyz="0 0 0" rpy="0 1.5707 1.5707"/>
       <mass value="5"/>
-      <cylinder_inertia m="5" r="0.1" h="0.05"/>
+      <cylinder_inertia m="5" r="0.03" h="0.02"/>
       <inertia
         ixx="1.0" ixy="0.0" ixz="0.0"
@@ -78,5 +56,5 @@
       <origin xyz="0 0 0" rpy="0 1.5707 1.5707"/>
       <geometry>
-        <cylinder radius="0.1" length="0.05"/>
+        <cylinder radius="0.03" length="0.02"/>
       </geometry>
     </collision>
@@ -84,5 +62,5 @@
       <origin xyz="0 0 0" rpy="0 1.5707 1.5707"/>
       <geometry>
-        <cylinder radius="0.1" length="0.05"/>
+        <cylinder radius="0.03" length="0.02"/>
       </geometry>
     </visual>
@@ -90,5 +68,5 @@
       <origin xyz="0 0 0" rpy="0 1.5707 1.5707"/>
       <mass value="5"/>
-      <cylinder_inertia m="5" r="0.1" h="0.05"/>
+      <cylinder_inertia m="5" r="0.03" h="0.02"/>
       <inertia
         ixx="1.0" ixy="0.0" ixz="0.0"
@@ -118,5 +96,5 @@
       <origin xyz="0 0 0" rpy="0 1.5707 1.5707"/>
       <geometry>
-        <cylinder radius="0.1" length="0.05"/>
+        <cylinder radius="0.03" length="0.02"/>
       </geometry>
     </collision>
@@ -124,5 +102,5 @@
       <origin xyz="0 0 0" rpy="0 1.5707 1.5707"/>
       <geometry>
-        <cylinder radius="0.1" length="0.05"/>
+        <cylinder radius="0.03" length="0.02"/>
       </geometry>
     </visual>
@@ -130,5 +108,5 @@
       <origin xyz="0 0 0" rpy="0 1.5707 1.5707"/>
       <mass value="5"/>
-      <cylinder_inertia m="5" r="0.1" h="0.05"/>
+      <cylinder_inertia m="5" r="0.03" h="0.02"/>
       <inertia
         ixx="1.0" ixy="0.0" ixz="0.0"
@@ -142,5 +120,5 @@
       <origin xyz="0 0 0" rpy="0 1.5707 1.5707"/>
       <geometry>
-        <cylinder radius="0.1" length="0.05"/>
+        <cylinder radius="0.03" length="0.02"/>
       </geometry>
     </collision>
@@ -148,5 +126,5 @@
       <origin xyz="0 0 0" rpy="0 1.5707 1.5707"/>
       <geometry>
-        <cylinder radius="0.1" length="0.05"/>
+        <cylinder radius="0.03" length="0.02"/>
       </geometry>
     </visual>
@@ -154,5 +132,5 @@
       <origin xyz="0 0 0" rpy="0 1.5707 1.5707"/>
       <mass value="5"/>
-      <cylinder_inertia m="5" r="0.1" h="0.05"/>
+      <cylinder_inertia m="5" r="0.03" h="0.02"/>
       <inertia
         ixx="1.0" ixy="0.0" ixz="0.0"

Commit message: Laser, mapping and amcl working

File: src/callisto_description/urdf/callisto.xacro (robot description, xacro)
@@ -13,5 +13,5 @@
       <inertia
           ixx="0.5" ixy="0" ixz="0"
-          iyy="1.0" iyz="0"
+          iyy="0.1" iyz="0"
           izz="0.1"
       />
@@ -19,5 +19,5 @@
     <collision name='collision'>
       <geometry>
-        <box size=".4 .2 .05"/>
+        <box size=".4 .2 .1"/>
       </geometry>
     </collision>
@@ -30,5 +30,5 @@
     </link>
   <link name="fleft_wheel">
-    <!--origin xyz="-0.1 0.13 0.1" rpy="0 1.5707 1.5707"/-->
+    <!--origin xyz="-0.1 0.13 -0.05" rpy="0 1.5707 1.5707"/-->
     <collision name="collision">
       <origin xyz="0 0 0" rpy="0 1.5707 1.5707"/>
@@ -54,5 +54,5 @@
   </link>
   <link name="fright_wheel">
-    <!--origin xyz="-0.1 -0.13 0.1" rpy="0 1.5707 1.5707"/-->
+    <!--origin xyz="-0.1 -0.13 -.05" rpy="0 1.5707 1.5707"/-->
     <collision name="collision">
       <origin xyz="0 0 0" rpy="0 1.5707 1.5707"/>
@@ -78,5 +78,5 @@
   </link>
   <joint type="continuous" name="fleft_wheel_hinge">
-    <origin xyz="-0.1 0.15 0" rpy="0 0 0"/>
+    <origin xyz="-0.1 0.15 -0.05" rpy="0 0 0"/>
     <child link="fleft_wheel"/>
     <parent link="chassis"/>
@@ -86,5 +86,5 @@
   </joint>
   <joint type="continuous" name="fright_wheel_hinge">
-    <origin xyz="-0.1 -0.15 0" rpy="0 0 0"/>
+    <origin xyz="-0.1 -0.15 -0.05" rpy="0 0 0"/>
     <child link="fright_wheel"/>
     <parent link="chassis"/>
@@ -94,5 +94,5 @@
   </joint>
   <link name="left_wheel">
-    <!--origin xyz="0.1 0.13 0.1" rpy="0 1.5707 1.5707"/-->
+    <!--origin xyz="0.1 0.13 -.05" rpy="0 1.5707 1.5707"/-->
     <collision name="collision">
       <origin xyz="0 0 0" rpy="0 1.5707 1.5707"/>
@@ -118,5 +118,5 @@
   </link>
   <link name="right_wheel">
-    <!--origin xyz="0.1 -0.13 0.1" rpy="0 1.5707 1.5707"/-->
+    <!--origin xyz="0.1 -0.13 -.05" rpy="0 1.5707 1.5707"/-->
     <collision name="collision">
       <origin xyz="0 0 0" rpy="0 1.5707 1.5707"/>
@@ -142,5 +142,5 @@
   </link>
   <joint type="continuous" name="left_wheel_hinge">
-    <origin xyz="0.1 0.15 0" rpy="0 0 0"/>
+    <origin xyz="0.1 0.15 -.05" rpy="0 0 0"/>
     <child link="left_wheel"/>
     <parent link="chassis"/>
@@ -150,5 +150,5 @@
   </joint>
   <joint type="continuous" name="right_wheel_hinge">
-    <origin xyz="0.1 -0.15 0" rpy="0 0 0"/>
+    <origin xyz="0.1 -0.15 -.05" rpy="0 0 0"/>
     <child link="right_wheel"/>
     <parent link="chassis"/>

Commit message: URDF Changes

File: src/callisto_description/urdf/callisto.xacro (robot description, xacro)
@@ -6,4 +6,8 @@
   <xacro:property name="cameraSize" value="0.05"/>
   <xacro:property name="cameraMass" value="0.1"/>
+  <xacro:property name="wheelDistanceX" value="0.03"/>
+  <xacro:property name="wheelDistanceY" value="0.0"/>
+  <xacro:property name="wheelDistanceZ" value="0.0375"/>
+<!-- Robot Chassis -->
   <link name='chassis'>
     <pose>0 0 0.1 0 0 0</pose>
@@ -25,8 +29,25 @@
       <origin xyz="0 0 0" rpy=" 0 0 0"/>
       <geometry>
-        <box size=".4 .2 .1"/>
+        <mesh filename="package://callisto_description/meshes/chassis.stl" scale="0.9 0.9 0.8"/>
       </geometry>
     </visual>
     </link>
+<!-- Chassis Top -->
+  <link name='chassis_top'>
+    <pose>0 0 0.035 0 0 0</pose>
+    <visual name='chassis_top_visual'>
+      <origin xyz="0 0 0.035" rpy=" 0 0 0"/>
+      <geometry>
+        <mesh filename="package://callisto_description/meshes/top.stl" scale="0.8 0.8 0.8"/>
+      </geometry>
+    <material name="blue"/>
+    </visual>
+    </link>
+  <joint name="chassis_top_joint" type="fixed">
+    <origin xyz="0 0 0.035" rpy="0 0 0"/>
+    <parent link="chassis"/>
+    <child link="chassis_top"/>
+  </joint>
+<!-- Left Wheel -->
   <link name="fleft_wheel">
     <!--origin xyz="-0.1 0.13 -0.05" rpy="0 1.5707 1.5707"/-->
@@ -38,7 +59,7 @@
     </collision>
     <visual name="fleft_wheel_visual">
-      <origin xyz="0 0 0" rpy="0 1.5707 1.5707"/>
-      <geometry>
-        <cylinder radius="0.03" length="0.02"/>
+      <origin xyz="${wheelDistanceX} ${wheelDistanceY} ${wheelDistanceZ}" rpy="0 0 0"/>
+      <geometry>
+        <mesh filename="package://callisto_description/meshes/wheel.stl" scale="0.6 0.6 0.6"/>
       </geometry>
     </visual>
@@ -62,7 +83,7 @@
     </collision>
     <visual name="fright_wheel_visual">
-      <origin xyz="0 0 0" rpy="0 1.5707 1.5707"/>
-      <geometry>
-        <cylinder radius="0.03" length="0.02"/>
+      <origin xyz="${wheelDistanceX} ${wheelDistanceY} ${wheelDistanceZ}" rpy="0 0 0"/>
+      <geometry>
+        <mesh filename="package://callisto_description/meshes/wheel.stl" scale="0.6 0.6 0.6"/>
       </geometry>
     </visual>
@@ -102,7 +123,7 @@
     </collision>
     <visual name="left_wheel_visual">
-      <origin xyz="0 0 0" rpy="0 1.5707 1.5707"/>
-      <geometry>
-        <cylinder radius="0.03" length="0.02"/>
+      <origin xyz="${wheelDistanceX} ${wheelDistanceY} ${wheelDistanceZ}" rpy="0 0 0"/>
+      <geometry>
+        <mesh filename="package://callisto_description/meshes/wheel.stl" scale="0.6 0.6 0.6"/>
       </geometry>
     </visual>
@@ -126,7 +147,7 @@
     </collision>
     <visual name="right_wheel_visual">
-      <origin xyz="0 0 0" rpy="0 1.5707 1.5707"/>
-      <geometry>
-        <cylinder radius="0.03" length="0.02"/>
+      <origin xyz="${wheelDistanceX} ${wheelDistanceY} ${wheelDistanceZ}" rpy="0 0 0"/>
+      <geometry>
+        <mesh filename="package://callisto_description/meshes/wheel.stl" scale="0.6 0.6 0.6"/>
       </geometry>
     </visual>
@@ -210,3 +231,28 @@
     </inertial>
   </link>
+  <joint name="imu_joint" type="fixed">
+    <axis xyz="1 0 0"/> <!-- 0 1 0 -->
+    <origin xyz="0 0 0.19"/>
+    <parent link="chassis"/>
+    <child link="imu_link"/>
+  </joint>
+<link name="imu_link">
+  <inertial>
+    <mass value="0.001"/>
+    <origin rpy="0 0 0" xyz="0 0 0"/>
+    <inertia ixx="0.0001" ixy="0" ixz="0" iyy="0.000001" iyz="0" izz="0.0001"/>
+  </inertial>
+  <visual>
+    <origin rpy="0 0 0" xyz="0 0 0"/>
+    <geometry>
+      <box size="0.001 0.001 0.001"/>
+    </geometry>
+  </visual>
+  <collision>
+    <origin rpy="0 0 0" xyz="0 0 0"/>
+    <geometry>
+      <box size=".001 .001 .001"/>
+    </geometry>
+  </collision>
+</link>
 </robot>

Commit message: Adding weel hub

File: src/callisto_description/urdf/callisto.xacro (robot description, xacro)
@@ -74,4 +74,20 @@
     </inertial>
   </link>
+<!-- Front Left Wheel Hub -->
+<link name='fleft_wheel_hub'>
+    <pose>${wheelDistanceX} ${wheelDistanceY} ${wheelDistanceZ} 0 0 0</pose>
+    <visual name='fleft_wheel_hub_visual'>
+      <origin xyz="${wheelDistanceX} ${wheelDistanceY} ${wheelDistanceZ}" rpy=" 0 0 0"/>
+      <geometry>
+        <mesh filename="package://callisto_description/meshes/hub.stl" scale="0.5 0.5 0.5"/>
+      </geometry>
+    <material name="blue"/>
+    </visual>
+    </link>
+  <joint name="fleft_wheel_hub_joint" type="fixed">
+    <origin xyz="0 0 0" rpy="0 0 0"/>
+    <parent link="fleft_wheel"/>
+    <child link="fleft_wheel_hub"/>
+  </joint>
   <link name="fright_wheel">
     <!--origin xyz="-0.1 -0.13 -.05" rpy="0 1.5707 1.5707"/-->
@@ -98,4 +114,20 @@
     </inertial>
   </link>
+<!-- Front Right Wheel Hub -->
+<link name='fright_wheel_hub'>
+    <pose>${wheelDistanceX} ${wheelDistanceY} ${wheelDistanceZ} 0 0 0</pose>
+    <visual name='fright_wheel_hub_visual'>
+      <origin xyz="${wheelDistanceX} ${wheelDistanceY} ${wheelDistanceZ}" rpy=" 0 0 0"/>
+      <geometry>
+        <mesh filename="package://callisto_description/meshes/hub.stl" scale="0.5 0.5 0.5"/>
+      </geometry>
+    <material name="blue"/>
+    </visual>
+    </link>
+  <joint name="fright_wheel_hub_joint" type="fixed">
+    <origin xyz="0 0 0" rpy="0 0 0"/>
+    <parent link="fright_wheel"/>
+    <child link="fright_wheel_hub"/>
+  </joint>
   <joint type="continuous" name="fleft_wheel_hinge">
     <origin xyz="-0.1 0.15 -0.05" rpy="0 0 0"/>
@@ -138,4 +170,20 @@
     </inertial>
   </link>
+<!-- Left Wheel Hub -->
+<link name='left_wheel_hub'>
+    <pose>${wheelDistanceX} ${wheelDistanceY} ${wheelDistanceZ} 0 0 0</pose>
+    <visual name='left_wheel_hub_visual'>
+      <origin xyz="${wheelDistanceX} ${wheelDistanceY} ${wheelDistanceZ}" rpy=" 0 0 0"/>
+      <geometry>
+        <mesh filename="package://callisto_description/meshes/hub.stl" scale="0.5 0.5 0.5"/>
+      </geometry>
+    <material name="blue"/>
+    </visual>
+    </link>
+  <joint name="left_wheel_hub_joint" type="fixed">
+    <origin xyz="0 0 0" rpy="0 0 0"/>
+    <parent link="left_wheel"/>
+    <child link="left_wheel_hub"/>
+  </joint>
   <link name="right_wheel">
     <!--origin xyz="0.1 -0.13 -.05" rpy="0 1.5707 1.5707"/-->
@@ -162,4 +210,20 @@
     </inertial>
   </link>
+<!-- Right Wheel Hub -->
+<link name='right_wheel_hub'>
+    <pose>${wheelDistanceX} ${wheelDistanceY} ${wheelDistanceZ} 0 0 0</pose>
+    <visual name='right_wheel_hub_visual'>
+      <origin xyz="${wheelDistanceX} ${wheelDistanceY} ${wheelDistanceZ}" rpy=" 0 0 0"/>
+      <geometry>
+        <mesh filename="package://callisto_description/meshes/hub.stl" scale="0.5 0.5 0.5"/>
+      </geometry>
+    <material name="blue"/>
+    </visual>
+    </link>
+  <joint name="right_wheel_hub_joint" type="fixed">
+    <origin xyz="0 0 0" rpy="0 0 0"/>
+    <parent link="right_wheel"/>
+    <child link="right_wheel_hub"/>
+  </joint>
   <joint type="continuous" name="left_wheel_hinge">
     <origin xyz="0.1 0.15 -.05" rpy="0 0 0"/>
@@ -231,28 +295,3 @@
     </inertial>
   </link>
-  <joint name="imu_joint" type="fixed">
-    <axis xyz="1 0 0"/> <!-- 0 1 0 -->
-    <origin xyz="0 0 0.19"/>
-    <parent link="chassis"/>
-    <child link="imu_link"/>
-  </joint>
-<link name="imu_link">
-  <inertial>
-    <mass value="0.001"/>
-    <origin rpy="0 0 0" xyz="0 0 0"/>
-    <inertia ixx="0.0001" ixy="0" ixz="0" iyy="0.000001" iyz="0" izz="0.0001"/>
-  </inertial>
-  <visual>
-    <origin rpy="0 0 0" xyz="0 0 0"/>
-    <geometry>
-      <box size="0.001 0.001 0.001"/>
-    </geometry>
-  </visual>
-  <collision>
-    <origin rpy="0 0 0" xyz="0 0 0"/>
-    <geometry>
-      <box size=".001 .001 .001"/>
-    </geometry>
-  </collision>
-</link>
 </robot>
