Commit message: removed mesh

File: src/callisto_description/urdf/callisto.xacro (robot description, xacro)
@@ -6,8 +6,4 @@
   <xacro:property name="cameraSize" value="0.05"/>
   <xacro:property name="cameraMass" value="0.1"/>
-  <xacro:property name="wheelDistanceX" value="0.03"/>
-  <xacro:property name="wheelDistanceY" value="0.0"/>
-  <xacro:property name="wheelDistanceZ" value="0.0375"/>
-<!-- Robot Chassis -->
   <link name='chassis'>
     <pose>0 0 0.1 0 0 0</pose>
@@ -29,25 +25,8 @@
       <origin xyz="0 0 0" rpy=" 0 0 0"/>
       <geometry>
-        <mesh filename="package://callisto_description/meshes/chassis.stl" scale="0.9 0.9 0.8"/>
+        <box size=".4 .2 .1"/>
       </geometry>
     </visual>
     </link>
-<!-- Chassis Top -->
-  <link name='chassis_top'>
-    <pose>0 0 0.035 0 0 0</pose>
-    <visual name='chassis_top_visual'>
-      <origin xyz="0 0 0.035" rpy=" 0 0 0"/>
-      <geometry>
-        <mesh filename="package://callisto_description/meshes/top.stl" scale="0.8 0.8 0.8"/>
-      </geometry>
-    <material name="blue"/>
-    </visual>
-    </link>
-  <joint name="chassis_top_joint" type="fixed">
-    <origin xyz="0 0 0.035" rpy="0 0 0"/>
-    <parent link="chassis"/>
-    <child link="chassis_top"/>
-  </joint>
-<!-- Left Wheel -->
   <link name="fleft_wheel">
     <!--origin xyz="-0.1 0.13 -0.05" rpy="0 1.5707 1.5707"/-->
@@ -59,35 +38,19 @@
     </collision>
     <visual name="fleft_wheel_visual">
-      <origin xyz="${wheelDistanceX} ${wheelDistanceY} ${wheelDistanceZ}" rpy="0 0 0"/>
-      <geometry>
-        <mesh filename="package://callisto_description/meshes/wheel.stl" scale="0.6 0.6 0.6"/>
-      </geometry>
-    </visual>
-    <inertial>
-      <origin xyz="0 0 0" rpy="0 1.5707 1.5707"/>
-      <mass value="5"/>
-      <cylinder_inertia m="5" r="0.03" h="0.02"/>
-      <inertia
-        ixx="1.0" ixy="0.0" ixz="0.0"
-        iyy="1.0" iyz="0.0"
-        izz="1.0"/>
-    </inertial>
-  </link>
-<!-- Front Left Wheel Hub -->
-<link name='fleft_wheel_hub'>
-    <pose>${wheelDistanceX} ${wheelDistanceY} ${wheelDistanceZ} 0 0 0</pose>
-    <visual name='fleft_wheel_hub_visual'>
-      <origin xyz="${wheelDistanceX} ${wheelDistanceY} ${wheelDistanceZ}" rpy=" 0 0 0"/>
-      <geometry>
-        <mesh filename="package://callisto_description/meshes/hub.stl" scale="0.5 0.5 0.5"/>
-      </geometry>
-    <material name="blue"/>
-    </visual>
-    </link>
-  <joint name="fleft_wheel_hub_joint" type="fixed">
-    <origin xyz="0 0 0" rpy="0 0 0"/>
-    <parent link="fleft_wheel"/>
-    <child link="fleft_wheel_hub"/>
-  </joint>
+      <origin xyz="0 0 0" rpy="0 1.5707 1.5707"/>
+      <geometry>
+        <cylinder radius="0.03" length="0.02"/>
+      </geometry>
+    </visual>
+    <inertial>
+      <origin xyz="0 0 0" rpy="0 1.5707 1.5707"/>
+      <mass value="5"/>
+      <cylinder_inertia m="5" r="0.03" h="0.02"/>
+      <inertia
+        ixx="1.0" ixy="0.0" ixz="0.0"
+        iyy="1.0" iyz="0.0"
+        izz="1.0"/>
+    </inertial>
+  </link>
   <link name="fright_wheel">
     <!--origin xyz="-0.1 -0.13 -.05" rpy="0 1.5707 1.5707"/-->
@@ -99,35 +62,19 @@
     </collision>
     <visual name="fright_wheel_visual">
-      <origin xyz="${wheelDistanceX} ${wheelDistanceY} ${wheelDistanceZ}" rpy="0 0 0"/>
-      <geometry>
-        <mesh filename="package://callisto_description/meshes/wheel.stl" scale="0.6 0.6 0.6"/>
-      </geometry>
-    </visual>
-    <inertial>
-      <origin xyz="0 0 0" rpy="0 1.5707 1.5707"/>
-      <mass value="5"/>
-      <cylinder_inertia m="5" r="0.03" h="0.02"/>
-      <inertia
-        ixx="1.0" ixy="0.0" ixz="0.0"
-        iyy="1.0" iyz="0.0"
-        izz="1.0"/>
-    </inertial>
-  </link>
-<!-- Front Right Wheel Hub -->
-<link name='fright_wheel_hub'>
-    <pose>${wheelDistanceX} ${wheelDistanceY} ${wheelDistanceZ} 0 0 0</pose>
-    <visual name='fright_wheel_hub_visual'>
-      <origin xyz="${wheelDistanceX} ${wheelDistanceY} ${wheelDistanceZ}" rpy=" 0 0 0"/>
-      <geometry>
-        <mesh filename="package://callisto_description/meshes/hub.stl" scale="0.5 0.5 0.5"/>
-      </geometry>
-    <material name="blue"/>
-    </visual>
-    </link>
-  <joint name="fright_wheel_hub_joint" type="fixed">
-    <origin xyz="0 0 0" rpy="0 0 0"/>
-    <parent link="fright_wheel"/>
-    <child link="fright_wheel_hub"/>
-  </joint>
+      <origin xyz="0 0 0" rpy="0 1.5707 1.5707"/>
+      <geometry>
+        <cylinder radius="0.03" length="0.02"/>
+      </geometry>
+    </visual>
+    <inertial>
+      <origin xyz="0 0 0" rpy="0 1.5707 1.5707"/>
+      <mass value="5"/>
+      <cylinder_inertia m="5" r="0.03" h="0.02"/>
+      <inertia
+        ixx="1.0" ixy="0.0" ixz="0.0"
+        iyy="1.0" iyz="0.0"
+        izz="1.0"/>
+    </inertial>
+  </link>
   <joint type="continuous" name="fleft_wheel_hinge">
     <origin xyz="-0.1 0.15 -0.05" rpy="0 0 0"/>
@@ -155,35 +102,19 @@
     </collision>
     <visual name="left_wheel_visual">
-      <origin xyz="${wheelDistanceX} ${wheelDistanceY} ${wheelDistanceZ}" rpy="0 0 0"/>
-      <geometry>
-        <mesh filename="package://callisto_description/meshes/wheel.stl" scale="0.6 0.6 0.6"/>
-      </geometry>
-    </visual>
-    <inertial>
-      <origin xyz="0 0 0" rpy="0 1.5707 1.5707"/>
-      <mass value="5"/>
-      <cylinder_inertia m="5" r="0.03" h="0.02"/>
-      <inertia
-        ixx="1.0" ixy="0.0" ixz="0.0"
-        iyy="1.0" iyz="0.0"
-        izz="1.0"/>
-    </inertial>
-  </link>
-<!-- Left Wheel Hub -->
-<link name='left_wheel_hub'>
-    <pose>${wheelDistanceX} ${wheelDistanceY} ${wheelDistanceZ} 0 0 0</pose>
-    <visual name='left_wheel_hub_visual'>
-      <origin xyz="${wheelDistanceX} ${wheelDistanceY} ${wheelDistanceZ}" rpy=" 0 0 0"/>
-      <geometry>
-        <mesh filename="package://callisto_description/meshes/hub.stl" scale="0.5 0.5 0.5"/>
-      </geometry>
-    <material name="blue"/>
-    </visual>
-    </link>
-  <joint name="left_wheel_hub_joint" type="fixed">
-    <origin xyz="0 0 0" rpy="0 0 0"/>
-    <parent link="left_wheel"/>
-    <child link="left_wheel_hub"/>
-  </joint>
+      <origin xyz="0 0 0" rpy="0 1.5707 1.5707"/>
+      <geometry>
+        <cylinder radius="0.03" length="0.02"/>
+      </geometry>
+    </visual>
+    <inertial>
+      <origin xyz="0 0 0" rpy="0 1.5707 1.5707"/>
+      <mass value="5"/>
+      <cylinder_inertia m="5" r="0.03" h="0.02"/>
+      <inertia
+        ixx="1.0" ixy="0.0" ixz="0.0"
+        iyy="1.0" iyz="0.0"
+        izz="1.0"/>
+    </inertial>
+  </link>
   <link name="right_wheel">
     <!--origin xyz="0.1 -0.13 -.05" rpy="0 1.5707 1.5707"/-->
@@ -195,35 +126,19 @@
     </collision>
     <visual name="right_wheel_visual">
-      <origin xyz="${wheelDistanceX} ${wheelDistanceY} ${wheelDistanceZ}" rpy="0 0 0"/>
-      <geometry>
-        <mesh filename="package://callisto_description/meshes/wheel.stl" scale="0.6 0.6 0.6"/>
-      </geometry>
-    </visual>
-    <inertial>
-      <origin xyz="0 0 0" rpy="0 1.5707 1.5707"/>
-      <mass value="5"/>
-      <cylinder_inertia m="5" r="0.03" h="0.02"/>
-      <inertia
-        ixx="1.0" ixy="0.0" ixz="0.0"
-        iyy="1.0" iyz="0.0"
-        izz="1.0"/>
-    </inertial>
-  </link>
-<!-- Right Wheel Hub -->
-<link name='right_wheel_hub'>
-    <pose>${wheelDistanceX} ${wheelDistanceY} ${wheelDistanceZ} 0 0 0</pose>
-    <visual name='right_wheel_hub_visual'>
-      <origin xyz="${wheelDistanceX} ${wheelDistanceY} ${wheelDistanceZ}" rpy=" 0 0 0"/>
-      <geometry>
-        <mesh filename="package://callisto_description/meshes/hub.stl" scale="0.5 0.5 0.5"/>
-      </geometry>
-    <material name="blue"/>
-    </visual>
-    </link>
-  <joint name="right_wheel_hub_joint" type="fixed">
-    <origin xyz="0 0 0" rpy="0 0 0"/>
-    <parent link="right_wheel"/>
-    <child link="right_wheel_hub"/>
-  </joint>
+      <origin xyz="0 0 0" rpy="0 1.5707 1.5707"/>
+      <geometry>
+        <cylinder radius="0.03" length="0.02"/>
+      </geometry>
+    </visual>
+    <inertial>
+      <origin xyz="0 0 0" rpy="0 1.5707 1.5707"/>
+      <mass value="5"/>
+      <cylinder_inertia m="5" r="0.03" h="0.02"/>
+      <inertia
+        ixx="1.0" ixy="0.0" ixz="0.0"
+        iyy="1.0" iyz="0.0"
+        izz="1.0"/>
+    </inertial>
+  </link>
   <joint type="continuous" name="left_wheel_hinge">
     <origin xyz="0.1 0.15 -.05" rpy="0 0 0"/>
